File: src/4key pad.kicad_sch (KiCad schematic)
At the start: 7 parts, among them J1 OLED_128x32, SW1 RotaryEncoder_Switch_MP, U2 Raspberry_Pi_Pico

Commit message: Add files via upload
Connections:
- net rsw2 is gone; now on net GND: SW1.S2, U2.3 (GND)
- net GND: now also U2.13 (GND), U2.23 (GND), U2.28 (GND), U2.38 (GND), U2.42 (GND)
